File: electronics/USB_plug/USB_plug.kicad_sch (KiCad schematic)
At the start: 4 parts, among them J1 Conn_01x06_Pin, P1 USB_C_Plug

Commit message: various improvements. Both pd_logger and power_meter fully functional
Other:
- note added: "USB-C plug breakout"
Changed lines of the file:
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@@
 	(generator_version "9.0")
 	(paper "A4")
+	(text "USB-C plug breakout"
+		(exclude_from_sim no)
+		(at 148.336 30.988 0)
+		(effects
+			(font
+				(size 5.08 5.08)
+				(thickness 1.016)
+				(bold yes)
+			)
+		)
+	)
 	(text "D+"
 		(exclude_from_sim no)
